File: Adafruit RP2040 Tester Brains rev A.kicad_pcb (KiCad board)
At the start: 2 copper layers, 69.9 x 104 mm, 48 parts, among them IC1 WS2811-SOP8, Q1 DMG34x5, Q2 DMG34x5, Q3 BSS138, Q4 BSS138, Q5 BSS138, SW1 12mm SMT, SW2 DPDT SLIDE, X1 USB A, X2 MicroSD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

Commit message: More migration to kKiCAD
Parts:
- removed JP8: , Adafruit RP2040 Tester Brains rev A:1X12_OVAL
- removed SP1: SPEAKER/PS12, Adafruit RP2040 Tester Brains rev A:PS12
- removed X2: MicroSD, Adafruit RP2040 Tester Brains rev A:MICROSD
- added C1: 10uF, Capacitor_SMD:C_0805_2012Metric_Pad1.18x1.45mm_HandSolder, F.Cu at (179.1, 88.8)
- added C2: 10uF, Capacitor_SMD:C_0805_2012Metric_Pad1.18x1.45mm_HandSolder, F.Cu at (179.1, 91.8)
- added C3: 10uF, Capacitor_SMD:C_0805_2012Metric_Pad1.18x1.45mm_HandSolder, F.Cu at (179.1, 94.8)
- added C4: 10uF, Capacitor_SMD:C_0805_2012Metric_Pad1.18x1.45mm_HandSolder, F.Cu at (179.1, 97.8)
- added C5: 10uF, Capacitor_SMD:C_0805_2012Metric_Pad1.18x1.45mm_HandSolder, F.Cu at (179.1, 100.9)
- added C6: 10uF, Capacitor_SMD:C_0805_2012Metric_Pad1.18x1.45mm_HandSolder, F.Cu at (179.1, 103.9)
- added C7: 10uF, Capacitor_SMD:C_0805_2012Metric_Pad1.18x1.45mm_HandSolder, F.Cu at (179.1, 106.9)
- added C8: 10uF, Capacitor_SMD:C_0805_2012Metric_Pad1.18x1.45mm_HandSolder, F.Cu at (179.1, 109.9)
- added C9: 10uF, Capacitor_SMD:C_0805_2012Metric_Pad1.18x1.45mm_HandSolder, F.Cu at (179.1, 112.9)
- added DS102: WC1602A, Display:WC1602A, F.Cu at (103.0, 62.0)
- added FID1: FIDUCIAL_1MM, Fiducial:Fiducial_1mm_Mask3mm, F.Cu at (177.1, 133.1)
- added FID2: FIDUCIAL_1MM, Fiducial:Fiducial_1mm_Mask3mm, F.Cu at (177.1, 137.7)
- added FID3: FIDUCIAL_1MM, Fiducial:Fiducial_1mm_Mask3mm, F.Cu at (177.1, 142.2)
- added J102: Micro_SD_Card_Det1, Connector_Card:microSD_HC_Molex_104031-0811, F.Cu at (133.2, 113.1)
- added J103: Conn_01x12, Connector_PinHeader_2.54mm:PinHeader_1x12_P2.54mm_Horizontal, F.Cu at (133.4, 145.7)
- added LS101: Speaker, Buzzer_Beeper:Buzzer_12x9.5RM7.6, F.Cu at (114.1, 110.6)
- added Q101: BSS138, Package_TO_SOT_SMD:SOT-23, F.Cu at (149.5, 107.6)
- added Q102: BSS138, Package_TO_SOT_SMD:SOT-23, F.Cu at (151.5, 119.0)
- added Q103: DMG2301L, Package_TO_SOT_SMD:SOT-23, F.Cu at (151.4, 127.7)
- added Q104: DMG2301L, Package_TO_SOT_SMD:SOT-23, F.Cu at (150.4, 136.1)
- added R1: 10K, Resistor_SMD:R_0603_1608Metric_Pad0.98x0.95mm_HandSolder, F.Cu at (175.5, 118.0)
- added R2: 10K, Resistor_SMD:R_0603_1608Metric_Pad0.98x0.95mm_HandSolder, F.Cu at (175.5, 120.5)
- added R3: 10K, Resistor_SMD:R_0603_1608Metric_Pad0.98x0.95mm_HandSolder, F.Cu at (175.5, 123.0)
- added R4: 10K, Resistor_SMD:R_0603_1608Metric_Pad0.98x0.95mm_HandSolder, F.Cu at (175.5, 125.5)
- added R5: 10K, Resistor_SMD:R_0603_1608Metric_Pad0.98x0.95mm_HandSolder, F.Cu at (175.5, 128.0)
- added SW102: SW_DPDT_x2, Button_Switch_THT:SW_CK_JS202011AQN_DPDT_Angled, F.Cu at (159.1, 145.9)
- added TP1: SEWTAP_SMTNUTM3, Adafruit RP2040 Tester Brains rev A:SMT_NUT_3MM, F.Cu at (173.1, 90.9)
- added TP2: SEWTAP_SMTNUTM3, Adafruit RP2040 Tester Brains rev A:SMT_NUT_3MM, F.Cu at (173.1, 98.2)
- added TP3: SEWTAP_SMTNUTM3, Adafruit RP2040 Tester Brains rev A:SMT_NUT_3MM, F.Cu at (173.1, 105.4)
- added TP4: SEWTAP_SMTNUTM3, Adafruit RP2040 Tester Brains rev A:SMT_NUT_3MM, F.Cu at (173.1, 112.7)
- added U$10: MOUNTINGHOLE3.0THIN, MountingHole:MountingHole_3.2mm_M3, F.Cu at (148.1, 175.0)
- added U$7: MOUNTINGHOLE3.0THIN, MountingHole:MountingHole_3.2mm_M3, F.Cu at (148.1, 151.1)
- added U$8: MOUNTINGHOLE3.0THIN, MountingHole:MountingHole_3.2mm_M3, F.Cu at (148.1, 159.1)
- added U$9: MOUNTINGHOLE3.0THIN, MountingHole:MountingHole_3.2mm_M3, F.Cu at (148.1, 167.0)
- added U101: WS2811, Package_SO:SOIC-8_3.9x4.9mm_P1.27mm, F.Cu at (179.0, 147.8)
- added VR101: 10K Trimmer, Adafruit RP2040 Tester Brains rev A:TRIMPOT_BOURNS_TC33X-2, F.Cu at (85.9, 41.7)
- moved CB1 0.34 mm to (124.9, 79.0)
Connections:
- net N$1 renamed /SPEAKER
- net SD_CD renamed /SD_CD
- CB1 pad S1: TXD -> /TXD
- CB1 pad S10: SWCLK -> /SWCLK
- CB1 pad S11: SDA -> /SDA
- CB1 pad S12: SDA -> /SDA
- CB1 pad S13: SCL -> /SCL
- CB1 pad S14: SCL -> /SCL
- CB1 pad S17: VBAT_SW -> /VBAT_SW
- CB1 pad S18: VBAT_SW -> /VBAT_SW
- CB1 pad S19: LCD_RS -> /LCD_RS
- CB1 pad S2: TXD -> /TXD
- CB1 pad S20: LCD_RS -> /LCD_RS
- CB1 pad S21: LCD_E -> /LCD_E
- CB1 pad S22: LCD_E -> /LCD_E
- CB1 pad S23: LCD_D4 -> /LCD_D4
- CB1 pad S24: LCD_D4 -> /LCD_D4
- CB1 pad S27: LCD_D5 -> /LCD_D5
- CB1 pad S28: LCD_D5 -> /LCD_D5
- CB1 pad S29: LCD_D6 -> /LCD_D6
- CB1 pad S3: RXD -> /RXD
- CB1 pad S30: LCD_D6 -> /LCD_D6
- CB1 pad S31: LCD_D7 -> /LCD_D7
- CB1 pad S32: LCD_D7 -> /LCD_D7
- CB1 pad S33: LCD_NEO -> /LCD_NEO
- CB1 pad S34: LCD_NEO -> /LCD_NEO
- CB1 pad S4: RXD -> /RXD
- CB1 pad S41: MISO -> /MISO
- CB1 pad S42: MISO -> /MISO
- CB1 pad S43: SD_CS -> /SD_CS
- CB1 pad S44: SD_CS -> /SD_CS
- CB1 pad S47: SCK -> /SCK
- CB1 pad S48: SCK -> /SCK
- CB1 pad S49: MOSI -> /MOSI
- CB1 pad S50: MOSI -> /MOSI
- CB1 pad S51: USB_D+ -> /USB_D+
- CB1 pad S52: USB_D+ -> /USB_D+
- CB1 pad S53: USB_D- -> /USB_D-
- CB1 pad S54: USB_D- -> /USB_D-
- CB1 pad S57: VUSB_SW -> /VUSB_SW
- CB1 pad S58: VUSB_SW -> /VUSB_SW
- CB1 pad S59: RESET -> /RESET
- CB1 pad S60: RESET -> /RESET
- CB1 pad S61: VMEAS_DIV2 -> /VMEAS_DIV2
- CB1 pad S62: VMEAS_DIV2 -> /VMEAS_DIV2
- CB1 pad S63: TARGET_RESET -> /TARGET_RESET
- CB1 pad S64: TARGET_RESET -> /TARGET_RESET
- CB1 pad S67: GPIO28 -> /GPIO28
- CB1 pad S68: GPIO28 -> /GPIO28
- CB1 pad S69: (no net) -> unconnected-(CB1-ADC_VREF-PadS69)
- CB1 pad S7: SWDIO -> /SWDIO
- CB1 pad S70: (no net) -> unconnected-(CB1-ADC_VREF-PadS69)_0
- CB1 pad S73: (no net) -> unconnected-(CB1-3.3V_EN-PadS73)_0
- CB1 pad S74: (no net) -> unconnected-(CB1-3.3V_EN-PadS73)
- CB1 pad S77: VSYS -> unconnected-(CB1-VSYS-PadS77)
- CB1 pad S78: VSYS -> unconnected-(CB1-VSYS-PadS77)_0
- CB1 pad S8: SWDIO -> /SWDIO
- CB1 pad S9: SWCLK -> /SWCLK
